File: kicad/clock.kicad_sch (KiCad schematic)
At the start: 5 parts, among them U8 74AUC2G240, Y2 SG-210STF

Commit message: finish schematic and almost done pcb routing
Parts:
- C26: renamed from C24; footprint (none) -> Capacitor_SMD:C_0402_1005Metric
- R13: renamed from R10; footprint (none) -> Resistor_SMD:R_0402_1005Metric
- R14: renamed from R21; footprint (none) -> Resistor_SMD:R_0402_1005Metric
- U5: renamed from U8; footprint (none) -> Package_SO:VSSOP-8_3x3mm_P0.65mm
- renumbered Y2 to Y1
Connections:
- net 12MHz_OUT renamed CLK_12M_OUT
Changed lines of the file:
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@@
 		)
 	)
-	(global_label "12MHz_OUT"
+	(hierarchical_label "CLK_12M_OUT"
 		(shape input)
 		(at 93.98 72.39 0)
-		(fields_autoplaced yes)
 		(effects
 			(font
@@
 			(justify left)
 		)
-		(property "Intersheetrefs" "${INTERSHEET_REFS}"
-			(at 107.7904 72.39 0)
-			(hide yes)
-			(show_name no)
-			(do_not_autoplace no)
-			(effects
-				(font
-					(size 1.27 1.27)
-				)
-				(justify left)
-			)
-		)
-	)
-	(global_label "IOB_25b_G3"
+	)
+	(hierarchical_label "IOB_25b_G3"
 		(shape input)
 		(at 100.33 49.53 0)
-		(fields_autoplaced yes)
 		(effects
 			(font
@@
 			)
 			(justify left)
-		)
-		(property "Intersheetrefs" "${INTERSHEET_REFS}"
-			(at 114.5032 49.53 0)
-			(hide yes)
-			(show_name no)
-			(do_not_autoplace no)
-			(effects
-				(font
-					(size 1.27 1.27)
-				)
-				(justify left)
-			)
 		)
 	)
@@
 		(dnp no)
 		(fields_autoplaced yes)
-		(property "Reference" "R21"
+		(property "Reference" "R14"
 			(at 96.52 43.18 90)
 			(show_name no)
@@
 			)
 		)
-		(property "Footprint" ""
+		(property "Footprint" "Resistor_SMD:R_0402_1005Metric"
 			(at 96.52 49.53 0)
 			(hide yes)
@@
 			(project "FPGA_Board"
 				(path "/ed5fd1e9-0492-49f2-b736-bd16e22cfa0b/b28031e3-dbc0-406e-8faf-efb7f86de153"
-					(reference "R21")
+					(reference "R14")
 					(unit 1)
 				)
@@
 		(dnp no)
 		(fields_autoplaced yes)
-		(property "Reference" "U8"
+		(property "Reference" "U5"
 			(at 78.74 81.28 0)
 			(show_name no)
@@
 			)
 		)
-		(property "Footprint" ""
+		(property "Footprint" "Package_SO:VSSOP-8_3x3mm_P0.65mm"
 			(at 80.01 72.39 0)
 			(hide yes)
@@
 			(project "FPGA_Board"
 				(path "/ed5fd1e9-0492-49f2-b736-bd16e22cfa0b/b28031e3-dbc0-406e-8faf-efb7f86de153"
-					(reference "U8")
+					(reference "U5")
 					(unit 1)
 				)
@@
 		(dnp yes)
 		(fields_autoplaced yes)
-		(property "Reference" "R10"
+		(property "Reference" "R13"
 			(at 35.56 63.4999 0)
 			(show_name no)
@@
 			)
 		)
-		(property "Footprint" ""
+		(property "Footprint" "Resistor_SMD:R_0402_1005Metric"
 			(at 33.02 64.77 0)
 			(hide yes)
@@
 			(project "FPGA_Board"
 				(path "/ed5fd1e9-0492-49f2-b736-bd16e22cfa0b/b28031e3-dbc0-406e-8faf-efb7f86de153"
-					(reference "R10")
+					(reference "R13")
 					(unit 1)
 				)
@@
 		(dnp no)
 		(fields_autoplaced yes)
-		(property "Reference" "#PWR041"
+		(property "Reference" "#PWR028"
 			(at 49.53 54.61 0)
 			(hide yes)
@@
 			(project "FPGA_Board"
 				(path "/ed5fd1e9-0492-49f2-b736-bd16e22cfa0b/b28031e3-dbc0-406e-8faf-efb7f86de153"
-					(reference "#PWR041")
+					(reference "#PWR028")
 					(unit 1)
 				)
@@
 		(dnp no)
 		(fields_autoplaced yes)
-		(property "Reference" "C24"
+		(property "Reference" "C26"
 			(at 52.07 43.1862 0)
 			(show_name no)
@@
 			)
 		)
-		(property "Footprint" ""
+		(property "Footprint" "Capacitor_SMD:C_0402_1005Metric"
 			(at 49.53 44.45 0)
 			(hide yes)
@@
 			(project "FPGA_Board"
 				(path "/ed5fd1e9-0492-49f2-b736-bd16e22cfa0b/b28031e3-dbc0-406e-8faf-efb7f86de153"
-					(reference "C24")
+					(reference "C26")
 					(unit 1)
 				)
@@
 		(in_pos_files yes)
 		(dnp no)
-		(property "Reference" "U8"
+		(property "Reference" "U5"
 			(at 78.74 40.64 0)
 			(show_name no)
@@
 			)
 		)
-		(property "Footprint" ""
+		(property "Footprint" "Package_SO:VSSOP-8_3x3mm_P0.65mm"
 			(at 80.01 49.53 0)
 			(hide yes)
@@
 			(project "FPGA_Board"
 				(path "/ed5fd1e9-0492-49f2-b736-bd16e22cfa0b/b28031e3-dbc0-406e-8faf-efb7f86de153"
-					(reference "U8")
+					(reference "U5")
 					(unit 2)
 				)
@@
 		(dnp no)
 		(fields_autoplaced yes)
-		(property "Reference" "Y2"
+		(property "Reference" "Y1"
 			(at 57.15 54.5398 0)
 			(show_name no)
@@
 			(project "FPGA_Board"
 				(path "/ed5fd1e9-0492-49f2-b736-bd16e22cfa0b/b28031e3-dbc0-406e-8faf-efb7f86de153"
-					(reference "Y2")
+					(reference "Y1")
 					(unit 1)
 				)
@@
 		(dnp no)
 		(fields_autoplaced yes)
-		(property "Reference" "#PWR039"
+		(property "Reference" "#PWR027"
 			(at 45.72 77.47 0)
 			(hide yes)
@@
 			(project "FPGA_Board"
 				(path "/ed5fd1e9-0492-49f2-b736-bd16e22cfa0b/b28031e3-dbc0-406e-8faf-efb7f86de153"
-					(reference "#PWR039")
+					(reference "#PWR027")
 					(unit 1)
 				)
@@
 		(dnp no)
 		(fields_autoplaced yes)
-		(property "Reference" "#PWR045"
+		(property "Reference" "#PWR029"
 			(at 72.39 60.96 0)
 			(hide yes)
@@
 			(project "FPGA_Board"
 				(path "/ed5fd1e9-0492-49f2-b736-bd16e22cfa0b/b28031e3-dbc0-406e-8faf-efb7f86de153"
-					(reference "#PWR045")
+					(reference "#PWR029")
 					(unit 1)
 				)
