File: kicad/config.kicad_sch (KiCad schematic)
At the start: 3 parts

Commit message: finish schematic and almost done pcb routing
Parts:
- R15: renamed from R18; value 0 -> 0R; footprint (none) -> Resistor_SMD:R_0402_1005Metric
- R16, R17: value 0 -> 0R; footprint (none) -> Resistor_SMD:R_0402_1005Metric
Changed lines of the file:
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@@
 		)
 	)
-	(global_label "IOB_22a"
+	(hierarchical_label "USB_D+"
+		(shape input)
+		(at 43.18 38.1 180)
+		(effects
+			(font
+				(size 1.27 1.27)
+			)
+			(justify right)
+		)
+	)
+	(hierarchical_label "IOB_22a"
 		(shape input)
 		(at 62.23 30.48 0)
-		(fields_autoplaced yes)
 		(effects
 			(font
@@
 			(justify left)
 		)
-		(property "Intersheetrefs" "${INTERSHEET_REFS}"
-			(at 72.9561 30.48 0)
-			(hide yes)
-			(show_name no)
-			(do_not_autoplace no)
-			(effects
-				(font
-					(size 1.27 1.27)
-				)
-				(justify left)
-			)
-		)
-	)
-	(global_label "IOB_23b"
+	)
+	(hierarchical_label "IOB_23b"
 		(shape input)
 		(at 62.23 38.1 0)
-		(fields_autoplaced yes)
 		(effects
 			(font
@@
 			(justify left)
 		)
-		(property "Intersheetrefs" "${INTERSHEET_REFS}"
-			(at 72.9561 38.1 0)
-			(hide yes)
-			(show_name no)
-			(do_not_autoplace no)
-			(effects
-				(font
-					(size 1.27 1.27)
-				)
-				(justify left)
-			)
-		)
-	)
-	(global_label "IOB_24a"
+	)
+	(hierarchical_label "USB_D-"
+		(shape input)
+		(at 43.18 43.18 180)
+		(effects
+			(font
+				(size 1.27 1.27)
+			)
+			(justify right)
+		)
+	)
+	(hierarchical_label "IOB_24a"
 		(shape input)
 		(at 62.23 43.18 0)
-		(fields_autoplaced yes)
 		(effects
 			(font
@@
 			)
 			(justify left)
-		)
-		(property "Intersheetrefs" "${INTERSHEET_REFS}"
-			(at 72.9561 43.18 0)
-			(hide yes)
-			(show_name no)
-			(do_not_autoplace no)
-			(effects
-				(font
-					(size 1.27 1.27)
-				)
-				(justify left)
-			)
-		)
-	)
-	(hierarchical_label "USB_D+"
-		(shape input)
-		(at 43.18 38.1 180)
-		(effects
-			(font
-				(size 1.27 1.27)
-			)
-			(justify right)
-		)
-	)
-	(hierarchical_label "USB_D-"
-		(shape input)
-		(at 43.18 43.18 180)
-		(effects
-			(font
-				(size 1.27 1.27)
-			)
-			(justify right)
 		)
 	)
@@
 			)
 		)
-		(property "Value" "0"
+		(property "Value" "0R"
 			(at 59.436 40.386 90)
 			(show_name no)
@@
 			)
 		)
-		(property "Footprint" ""
+		(property "Footprint" "Resistor_SMD:R_0402_1005Metric"
 			(at 57.15 43.18 0)
 			(hide yes)
@@
 		(dnp yes)
 		(fields_autoplaced yes)
-		(property "Reference" "R18"
+		(property "Reference" "R15"
 			(at 46.99 33.0199 0)
 			(show_name no)
@@
 			)
 		)
-		(property "Value" "0"
+		(property "Value" "0R"
 			(at 46.99 35.5599 0)
 			(show_name no)
@@
 			)
 		)
-		(property "Footprint" ""
+		(property "Footprint" "Resistor_SMD:R_0402_1005Metric"
 			(at 44.45 34.29 0)
 			(hide yes)
@@
 			(project "FPGA_Board"
 				(path "/ed5fd1e9-0492-49f2-b736-bd16e22cfa0b/04b4845f-9dd8-4013-ba5e-71062b138c05"
-					(reference "R18")
+					(reference "R15")
 					(unit 1)
 				)
@@
 			)
 		)
-		(property "Value" "0"
+		(property "Value" "0R"
 			(at 59.436 35.814 90)
 			(show_name no)
@@
 			)
 		)
-		(property "Footprint" ""
+		(property "Footprint" "Resistor_SMD:R_0402_1005Metric"
 			(at 57.15 38.1 0)
 			(hide yes)
