File: kicad/headers.kicad_sch (KiCad schematic)
At the start: 1 part, among them J3 Conn_02x24_Odd_Even

Commit message: finish schematic and almost done pcb routing
Parts:
- removed J3: Conn_02x24_Odd_Even, Connector_PinHeader_2.54mm:PinHeader_2x24_P2.54mm_Vertical, symbol Connector_Generic:Conn_02x24_Odd_Even
- added J3, J4: Conn_02x12_Odd_Even, Connector_PinHeader_2.54mm:PinHeader_2x12_P2.54mm_Vertical, symbol Connector_Generic:Conn_02x12_Odd_Even
Connections:
- net 3.3V: now also J3.22 (Pin_22), J3.23 (Pin_23)
- net CDONE: now also J4.6 (Pin_6)
- net CRESET: now also J4.5 (Pin_5)
- net FPGA_SI: now also J3.5 (Pin_5)
- net FPGA_SO: now also J3.2 (Pin_2)
- net FT_CS: now also J3.4 (Pin_4)
- net FT_SCK: now also J3.3 (Pin_3)
- net GND: now also J3.21 (Pin_21), J3.24 (Pin_24), J4.23 (Pin_23), J4.24 (Pin_24)
- net IOB_0a: now also J4.13 (Pin_13)
- net IOB_13b: now also J4.7 (Pin_7)
- net IOB_16a: now also J4.4 (Pin_4)
- net IOB_18a: now also J4.3 (Pin_3)
- net IOB_20a: now also J4.2 (Pin_2)
- net IOB_22a: now also J4.1 (Pin_1)
- net IOB_23b: now also J3.9 (Pin_9)
- net IOB_24a: now also J3.1 (Pin_1)
- net IOB_25b_G3: now also J3.8 (Pin_8)
- net IOB_29b: now also J3.7 (Pin_7)
- net IOB_2a: now also J4.12 (Pin_12)
- net IOB_31b: now also J3.6 (Pin_6)
- net IOB_3b_G6: now also J4.15 (Pin_15)
- net IOB_4a: now also J4.11 (Pin_11)
- net IOB_5b: now also J4.14 (Pin_14)
- net IOB_6a: now also J4.10 (Pin_10)
- net IOB_8a: now also J4.8 (Pin_8)
- net IOB_9b: now also J4.9 (Pin_9)
- net IOT_36b: now also J3.11 (Pin_11)
- net IOT_37a: now also J3.10 (Pin_10)
- net IOT_38b: now also J3.13 (Pin_13)
- net IOT_39a: now also J3.12 (Pin_12)
- net IOT_41a: now also J3.14 (Pin_14)
- net IOT_42b: now also J3.15 (Pin_15)
- net IOT_43a: now also J3.16 (Pin_16)
- net IOT_44b: now also J3.17 (Pin_17)
- net IOT_45a_G1: now also J4.22 (Pin_22)
- net IOT_46b_G0: now also J3.18 (Pin_18)
- net IOT_48b: now also J3.19 (Pin_19)
- net IOT_49a: now also J4.16 (Pin_16)
- net IOT_50b: now also J4.21 (Pin_21)
- net IOT_51a: now also J4.17 (Pin_17)
- net RGB0: now also J4.20 (Pin_20)
- net RGB1: now also J4.19 (Pin_19)
- net RGB2: now also J4.18 (Pin_18)
- new net CLK_12M_OUT: J3.20 (Pin_20)
