File: kicad/FPGA_Board.kicad_sch (KiCad schematic)
At the start: 0 parts

Commit message: finish schematic and almost done pcb routing
Parts:
- added FID1, FID2, FID3, FID4: Fiducial, Fiducial:Fiducial_0.5mm_Mask1mm, symbol Mechanical:Fiducial
- added FID5: Fiducial, Fiducial:Fiducial_Cross_1.5mm_Mask2mm, symbol Mechanical:Fiducial
- added H1, H2, H3, H4: MountingHole, MountingHole:MountingHole_3.2mm_M3, symbol Mechanical:MountingHole
Other:
- sheet Clock ports: added CLK_12M_OUT, IOB_25b_G3; removed none
- sheet Config ports: added IOB_22a, IOB_23b, IOB_24a; removed none
- sheet Headers ports: added 3.3V, CDONE, CLK_12M_OUT, CRESET, FPGA_SI, FPGA_SO, FT_CS, FT_SCK, IOB_0a, IOB_13b, IOB_16a, IOB_18a, IOB_20a, IOB_22a, IOB_23b, IOB_24a, IOB_25b_G3, IOB_29b, IOB_2a, IOB_31b, IOB_3b_G6, IOB_4a, IOB_5b, IOB_6a, IOB_8a, IOB_9b, IOT_36b, IOT_37a, IOT_38b, IOT_39a, IOT_41a, IOT_42b, IOT_43a, IOT_44b, IOT_45a_G1, IOT_46b_G0, IOT_48b, IOT_49a, IOT_50b, IOT_51a, RGB0, RGB1, RGB2; removed none

Commit message: add images and render
Parts:
- removed FID5: Fiducial, Fiducial:Fiducial_Cross_1.5mm_Mask2mm, symbol Mechanical:Fiducial
Changed lines of the file:
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@@
-	)
-	(symbol
-		(lib_id "Mechanical:Fiducial")
-		(at 127 185.42 0)
-		(unit 1)
-		(body_style 1)
-		(exclude_from_sim no)
-		(in_bom no)
-		(on_board yes)
-		(in_pos_files yes)
-		(dnp no)
-		(fields_autoplaced yes)
-		(property "Reference" "FID5"
-			(at 129.54 184.1499 0)
-			(show_name no)
-			(do_not_autoplace no)
-			(effects
-				(font
-					(size 1.27 1.27)
-				)
-				(justify left)
-			)
-		)
-		(property "Value" "Fiducial"
-			(at 129.54 186.6899 0)
-			(show_name no)
-			(do_not_autoplace no)
-			(effects
-				(font
-					(size 1.27 1.27)
-				)
-				(justify left)
-			)
-		)
-		(property "Footprint" "Fiducial:Fiducial_Cross_1.5mm_Mask2mm"
-			(at 127 185.42 0)
-			(hide yes)
-			(show_name no)
-			(do_not_autoplace no)
-			(effects
-				(font
-					(size 1.27 1.27)
-				)
-			)
-		)
-		(property "Datasheet" ""
-			(at 127 185.42 0)
-			(hide yes)
-			(show_name no)
-			(do_not_autoplace no)
-			(effects
-				(font
-					(size 1.27 1.27)
-				)
-			)
-		)
-		(property "Description" "Fiducial Marker"
-			(at 127 185.42 0)
-			(hide yes)
-			(show_name no)
-			(do_not_autoplace no)
-			(effects
-				(font
-					(size 1.27 1.27)
-				)
-			)
-		)
-		(instances
-			(project "FPGA_Board"
-				(path "/ed5fd1e9-0492-49f2-b736-bd16e22cfa0b"
-					(reference "FID5")
-					(unit 1)
-				)
-			)
-		)
 	)
 	(symbol
