File: kicad/power.kicad_sch (KiCad schematic)
At the start: 17 parts, among them U3 TLV75712PDBV, U4 TLV75725PDBV, U5 TLV75733PDBV, U8 74AUC2G240

Commit message: finish schematic and almost done pcb routing
Parts:
- C10, C11, C12, C13, C14, C3, C4, C5, C6, C7, C8, C9: footprint (none) -> Capacitor_SMD:C_0402_1005Metric
- C15: renamed from C25; footprint (none) -> Capacitor_SMD:C_0402_1005Metric
- U5: renamed from U8; footprint (none) -> Package_SO:VSSOP-8_3x3mm_P0.65mm
- renumbered U3 to U2, U4 to U3, U5 to U4
Other:
- note added: "add led indicators"
Changed lines of the file:
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@@
 	(generator_version "10.0")
 	(paper "A4")
+	(text "add led indicators"
+		(exclude_from_sim no)
+		(at 58.4199 43.0914 0)
+		(effects
+			(font
+				(size 1.27 1.27)
+			)
+		)
+	)
 	(junction
 		(at 54.61 74.93)
@@
 			)
 		)
-		(property "Footprint" ""
+		(property "Footprint" "Capacitor_SMD:C_0402_1005Metric"
 			(at 54.61 66.04 0)
 			(hide yes)
@@
 		(dnp no)
 		(fields_autoplaced yes)
-		(property "Reference" "U4"
+		(property "Reference" "U3"
 			(at 43.18 57.15 0)
 			(show_name no)
@@
 			(project "FPGA_Board"
 				(path "/ed5fd1e9-0492-49f2-b736-bd16e22cfa0b/76f7b54c-e28b-4bc1-87b2-9b178c63eb5d"
-					(reference "U4")
+					(reference "U3")
 					(unit 1)
 				)
@@
 		(dnp no)
 		(fields_autoplaced yes)
-		(property "Reference" "#PWR043"
+		(property "Reference" "#PWR09"
 			(at 88.9 66.04 0)
 			(hide yes)
@@
 			(project "FPGA_Board"
 				(path "/ed5fd1e9-0492-49f2-b736-bd16e22cfa0b/76f7b54c-e28b-4bc1-87b2-9b178c63eb5d"
-					(reference "#PWR043")
+					(reference "#PWR09")
 					(unit 1)
 				)
@@
 			)
 		)
-		(property "Footprint" ""
+		(property "Footprint" "Capacitor_SMD:C_0402_1005Metric"
 			(at 64.77 27.94 0)
 			(hide yes)
@@
 			)
 		)
-		(property "Footprint" ""
+		(property "Footprint" "Capacitor_SMD:C_0402_1005Metric"
 			(at 15.24 27.94 0)
 			(hide yes)
@@
 			)
 		)
-		(property "Footprint" ""
+		(property "Footprint" "Capacitor_SMD:C_0402_1005Metric"
 			(at 64.77 66.04 0)
 			(hide yes)
@@
 		(dnp no)
 		(fields_autoplaced yes)
-		(property "Reference" "U8"
+		(property "Reference" "U5"
 			(at 95.25 46.9899 0)
 			(show_name no)
@@
 			)
 		)
-		(property "Footprint" ""
+		(property "Footprint" "Package_SO:VSSOP-8_3x3mm_P0.65mm"
 			(at 88.9 48.26 0)
 			(hide yes)
@@
 			(project "FPGA_Board"
 				(path "/ed5fd1e9-0492-49f2-b736-bd16e22cfa0b/76f7b54c-e28b-4bc1-87b2-9b178c63eb5d"
-					(reference "U8")
+					(reference "U5")
 					(unit 3)
 				)
@@
 		(dnp no)
 		(fields_autoplaced yes)
-		(property "Reference" "U3"
+		(property "Reference" "U2"
 			(at 43.18 19.05 0)
 			(show_name no)
@@
 			(project "FPGA_Board"
 				(path "/ed5fd1e9-0492-49f2-b736-bd16e22cfa0b/76f7b54c-e28b-4bc1-87b2-9b178c63eb5d"
-					(reference "U3")
+					(reference "U2")
 					(unit 1)
 				)
@@
 			)
 		)
-		(property "Footprint" ""
+		(property "Footprint" "Capacitor_SMD:C_0402_1005Metric"
 			(at 15.24 66.04 0)
 			(hide yes)
@@
 		(dnp no)
 		(fields_autoplaced yes)
-		(property "Reference" "C25"
+		(property "Reference" "C15"
 			(at 95.25 27.9462 0)
 			(show_name no)
@@
 			)
 		)
-		(property "Footprint" ""
+		(property "Footprint" "Capacitor_SMD:C_0402_1005Metric"
 			(at 92.71 29.21 0)
 			(hide yes)
@@
 			(project "FPGA_Board"
 				(path "/ed5fd1e9-0492-49f2-b736-bd16e22cfa0b/76f7b54c-e28b-4bc1-87b2-9b178c63eb5d"
-					(reference "C25")
+					(reference "C15")
 					(unit 1)
 				)
@@
 			)
 		)
-		(property "Footprint" ""
+		(property "Footprint" "Capacitor_SMD:C_0402_1005Metric"
 			(at 25.4 104.14 0)
 			(hide yes)
@@
 		(dnp no)
 		(fields_autoplaced yes)
-		(property "Reference" "#PWR044"
+		(property "Reference" "#PWR010"
 			(at 92.71 39.37 0)
 			(hide yes)
@@
 			(project "FPGA_Board"
 				(path "/ed5fd1e9-0492-49f2-b736-bd16e22cfa0b/76f7b54c-e28b-4bc1-87b2-9b178c63eb5d"
-					(reference "#PWR044")
+					(reference "#PWR010")
 					(unit 1)
 				)
@@
 		(dnp no)
 		(fields_autoplaced yes)
-		(property "Reference" "#PWR010"
+		(property "Reference" "#PWR08"
 			(at 43.18 120.65 0)
 			(hide yes)
@@
 			(project "FPGA_Board"
 				(path "/ed5fd1e9-0492-49f2-b736-bd16e22cfa0b/76f7b54c-e28b-4bc1-87b2-9b178c63eb5d"
-					(reference "#PWR010")
+					(reference "#PWR08")
 					(unit 1)
 				)
@@
 			)
 		)
-		(property "Footprint" ""
+		(property "Footprint" "Capacitor_SMD:C_0402_1005Metric"
 			(at 54.61 104.14 0)
 			(hide yes)
@@
 			)
 		)
-		(property "Footprint" ""
+		(property "Footprint" "Capacitor_SMD:C_0402_1005Metric"
 			(at 25.4 66.04 0)
 			(hide yes)
@@
 		(dnp no)
 		(fields_autoplaced yes)
-		(property "Reference" "U5"
+		(property "Reference" "U4"
 			(at 43.18 95.25 0)
 			(show_name no)
@@
 			(project "FPGA_Board"
 				(path "/ed5fd1e9-0492-49f2-b736-bd16e22cfa0b/76f7b54c-e28b-4bc1-87b2-9b178c63eb5d"
-					(reference "U5")
+					(reference "U4")
 					(unit 1)
 				)
@@
 			)
 		)
-		(property "Footprint" ""
+		(property "Footprint" "Capacitor_SMD:C_0402_1005Metric"
 			(at 64.77 104.14 0)
 			(hide yes)
@@
 		(dnp no)
 		(fields_autoplaced yes)
-		(property "Reference" "#PWR08"
+		(property "Reference" "#PWR06"
 			(at 43.18 44.45 0)
 			(hide yes)
@@
 			(project "FPGA_Board"
 				(path "/ed5fd1e9-0492-49f2-b736-bd16e22cfa0b/76f7b54c-e28b-4bc1-87b2-9b178c63eb5d"
-					(reference "#PWR08")
+					(reference "#PWR06")
 					(unit 1)
 				)
@@
 			)
 		)
-		(property "Footprint" ""
+		(property "Footprint" "Capacitor_SMD:C_0402_1005Metric"
 			(at 15.24 104.14 0)
 			(hide yes)
@@
 		(dnp no)
 		(fields_autoplaced yes)
-		(property "Reference" "#PWR09"
+		(property "Reference" "#PWR07"
 			(at 43.18 82.55 0)
 			(hide yes)
@@
 			(project "FPGA_Board"
 				(path "/ed5fd1e9-0492-49f2-b736-bd16e22cfa0b/76f7b54c-e28b-4bc1-87b2-9b178c63eb5d"
-					(reference "#PWR09")
+					(reference "#PWR07")
 					(unit 1)
 				)
@@
 			)
 		)
-		(property "Footprint" ""
+		(property "Footprint" "Capacitor_SMD:C_0402_1005Metric"
 			(at 54.61 27.94 0)
 			(hide yes)
@@
 			)
 		)
-		(property "Footprint" ""
+		(property "Footprint" "Capacitor_SMD:C_0402_1005Metric"
 			(at 25.4 27.94 0)
 			(hide yes)

Commit message: add images and render
Parts:
- added TP13, TP14, TP15: TestPoint, TestPoint:TestPoint_Pad_2.0x2.0mm, symbol Connector:TestPoint
Connections:
- net 1.2V: now also TP13.1
- net 2.5V: now also TP14.1
- net 3.3V: now also TP15.1

Commit message: update bom and journal
Connections:
- net 1.2V: now also U3.3 (EN)
- net 2.5V: now also U4.3 (EN)
- net VIN: no longer U3.3 (EN), U4.3 (EN)
Changed lines of the file:
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@@
-	)
-	(junction
-		(at 34.29 101.6)
-		(diameter 0)
-		(color 0 0 0 0)
 	)
 	(junction
@@
 	)
 	(junction
-		(at 34.29 63.5)
-		(diameter 0)
-		(color 0 0 0 0)
-	)
-	(junction
 		(at 64.77 63.5)
 		(diameter 0)
@@
 	(wire
 		(pts
-			(xy 34.29 66.04) (xy 34.29 63.5)
-		)
-		(stroke
-			(width 0)
-			(type default)
-		)
-	)
-	(wire
-		(pts
 			(xy 50.8 63.5) (xy 54.61 63.5)
 		)
@@
 	(wire
 		(pts
-			(xy 34.29 104.14) (xy 34.29 101.6)
-		)
-		(stroke
-			(width 0)
-			(type default)
-		)
-	)
-	(wire
-		(pts
 			(xy 15.24 30.48) (xy 15.24 36.83)
 		)
@@
 	(wire
 		(pts
-			(xy 34.29 63.5) (xy 35.56 63.5)
+			(xy 25.4 63.5) (xy 35.56 63.5)
 		)
 		(stroke
@@
 	(wire
 		(pts
-			(xy 25.4 63.5) (xy 34.29 63.5)
-		)
-		(stroke
-			(width 0)
-			(type default)
-		)
-	)
-	(wire
-		(pts
 			(xy 25.4 74.93) (xy 43.18 74.93)
 		)
@@
 	(wire
 		(pts
-			(xy 25.4 101.6) (xy 34.29 101.6)
+			(xy 25.4 101.6) (xy 35.56 101.6)
 		)
 		(stroke
@@
 	(wire
 		(pts
+			(xy 34.29 104.14) (xy 34.29 105.41)
+		)
+		(stroke
+			(width 0)
+			(type default)
+		)
+	)
+	(wire
+		(pts
 			(xy 64.77 106.68) (xy 64.77 113.03)
 		)
@@
 	(wire
 		(pts
-			(xy 34.29 101.6) (xy 35.56 101.6)
-		)
-		(stroke
-			(width 0)
-			(type default)
-		)
-	)
-	(wire
-		(pts
 			(xy 25.4 106.68) (xy 25.4 113.03)
 		)
@@
 		(pts
 			(xy 35.56 66.04) (xy 34.29 66.04)
+		)
+		(stroke
+			(width 0)
+			(type default)
+		)
+	)
+	(wire
+		(pts
+			(xy 34.29 66.04) (xy 34.29 67.31)
 		)
 		(stroke
@@
 		)
 	)
+	(hierarchical_label "2.5V"
+		(shape input)
+		(at 34.29 105.41 270)
+		(effects
+			(font
+				(size 1.27 1.27)
+			)
+			(justify right)
+		)
+	)
 	(hierarchical_label "3.3V"
 		(shape input)
@@
 		)
 	)
+	(hierarchical_label "1.2V"
+		(shape input)
+		(at 34.29 67.31 270)
+		(effects
+			(font
+				(size 1.27 1.27)
+			)
+			(justify right)
+		)
+	)
