File: kicad/usb.kicad_sch (KiCad schematic)
At the start: 9 parts, among them J1 USB_C_Receptacle_USB2.0_14P, U2 USBLC6-2SC6

Commit message: finish schematic and almost done pcb routing
Parts:
- C1: renamed from C34; footprint (none) -> Capacitor_SMD:C_0402_1005Metric
- C2: renamed from C33; footprint (none) -> Capacitor_SMD:C_0402_1005Metric
- FB1: renamed from FB3; footprint (none) -> Inductor_SMD:L_0603_1608Metric
- J1: footprint (none) -> Connector_USB:USB_C_Receptacle_HRO_TYPE-C-31-M-12
- R1, R2, R3, R4: footprint (none) -> Resistor_SMD:R_0402_1005Metric
- renumbered U2 to U1
Changed lines of the file:
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@@
 			)
 		)
-		(property "Footprint" ""
+		(property "Footprint" "Resistor_SMD:R_0402_1005Metric"
 			(at 81.28 50.8 0)
 			(hide yes)
@@
 		(dnp no)
 		(fields_autoplaced yes)
-		(property "Reference" "#PWR060"
+		(property "Reference" "#PWR02"
 			(at 60.96 21.59 0)
 			(hide yes)
@@
 			(project "FPGA_Board"
 				(path "/ed5fd1e9-0492-49f2-b736-bd16e22cfa0b/ddd0c691-6505-4095-8238-9a1e5535ce52"
-					(reference "#PWR060")
+					(reference "#PWR02")
 					(unit 1)
 				)
@@
 		(dnp no)
 		(fields_autoplaced yes)
-		(property "Reference" "C33"
+		(property "Reference" "C2"
 			(at 93.98 38.1062 0)
 			(show_name no)
@@
 			)
 		)
-		(property "Footprint" ""
+		(property "Footprint" "Capacitor_SMD:C_0402_1005Metric"
 			(at 91.44 39.37 0)
 			(hide yes)
@@
 			(project "FPGA_Board"
 				(path "/ed5fd1e9-0492-49f2-b736-bd16e22cfa0b/ddd0c691-6505-4095-8238-9a1e5535ce52"
-					(reference "C33")
+					(reference "C2")
 					(unit 1)
 				)
@@
 			)
 		)
-		(property "Footprint" ""
+		(property "Footprint" "Resistor_SMD:R_0402_1005Metric"
 			(at 74.93 40.64 0)
 			(hide yes)
@@
 		(dnp no)
 		(fields_autoplaced yes)
-		(property "Reference" "C34"
+		(property "Reference" "C1"
 			(at 58.42 33.0138 0)
 			(show_name no)
@@
 			)
 		)
-		(property "Footprint" ""
+		(property "Footprint" "Capacitor_SMD:C_0402_1005Metric"
 			(at 60.96 31.75 0)
 			(hide yes)
@@
 			(project "FPGA_Board"
 				(path "/ed5fd1e9-0492-49f2-b736-bd16e22cfa0b/ddd0c691-6505-4095-8238-9a1e5535ce52"
-					(reference "C34")
+					(reference "C1")
 					(unit 1)
 				)
@@
 		(in_pos_files yes)
 		(dnp no)
-		(property "Reference" "U2"
+		(property "Reference" "U1"
 			(at 56.388 45.72 0)
 			(show_name no)
@@
 			(project "FPGA_Board"
 				(path "/ed5fd1e9-0492-49f2-b736-bd16e22cfa0b/ddd0c691-6505-4095-8238-9a1e5535ce52"
-					(reference "U2")
+					(reference "U1")
 					(unit 1)
 				)
@@
 		(dnp no)
 		(fields_autoplaced yes)
-		(property "Reference" "FB3"
+		(property "Reference" "FB1"
 			(at 72.3519 29.21 90)
 			(show_name no)
@@
 			)
 		)
-		(property "Footprint" ""
+		(property "Footprint" "Inductor_SMD:L_0603_1608Metric"
 			(at 72.39 37.338 90)
 			(hide yes)
@@
 			(project "FPGA_Board"
 				(path "/ed5fd1e9-0492-49f2-b736-bd16e22cfa0b/ddd0c691-6505-4095-8238-9a1e5535ce52"
-					(reference "FB3")
+					(reference "FB1")
 					(unit 1)
 				)
@@
 		(dnp no)
 		(fields_autoplaced yes)
-		(property "Reference" "#PWR02"
+		(property "Reference" "#PWR01"
 			(at 38.1 82.55 0)
 			(hide yes)
@@
 			(project "FPGA_Board"
 				(path "/ed5fd1e9-0492-49f2-b736-bd16e22cfa0b/ddd0c691-6505-4095-8238-9a1e5535ce52"
-					(reference "#PWR02")
+					(reference "#PWR01")
 					(unit 1)
 				)
@@
 			)
 		)
-		(property "Footprint" ""
+		(property "Footprint" "Connector_USB:USB_C_Receptacle_HRO_TYPE-C-31-M-12"
 			(at 41.91 50.8 0)
 			(hide yes)
@@
 			)
 		)
-		(property "Footprint" ""
+		(property "Footprint" "Resistor_SMD:R_0402_1005Metric"
 			(at 74.93 53.34 0)
 			(hide yes)
@@
 			)
 		)
-		(property "Footprint" ""
+		(property "Footprint" "Resistor_SMD:R_0402_1005Metric"
 			(at 68.58 43.18 0)
 			(hide yes)
@@
 		(dnp no)
 		(fields_autoplaced yes)
-		(property "Reference" "#PWR058"
+		(property "Reference" "#PWR05"
 			(at 91.44 49.53 0)
 			(hide yes)
@@
 			(project "FPGA_Board"
 				(path "/ed5fd1e9-0492-49f2-b736-bd16e22cfa0b/ddd0c691-6505-4095-8238-9a1e5535ce52"
-					(reference "#PWR058")
-					(unit 1)
-				)
+					(reference "#PWR05")
+					(unit 1)
+				)

Commit message: update bom and journal
Parts:
- added C37: 0.1uF, Capacitor_SMD:C_0402_1005Metric, symbol Device:C_Small
- R3, R4: value 5.1k -> 22
Connections:
- net GND: now also C37.2
- net at C1.1, FB1.1, J1.A4 (VBUS)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: now also C37.1
Other:
- moved on the sheet: C2, FB1, R1, R2, R3, R4
