File: kicad/flasher.kicad_sch (KiCad schematic)
At the start: 30 parts, among them U1 FT232H, U9 93LC56BT-I/OT

Commit message: finish schematic and almost done pcb routing
Parts:
- C27: renamed from C32; footprint (none) -> Capacitor_SMD:C_0402_1005Metric
- C28: renamed from C31; footprint (none) -> Capacitor_SMD:C_0402_1005Metric
- C29: renamed from C1; footprint (none) -> Capacitor_SMD:C_0402_1005Metric
- C30: renamed from C2; footprint (none) -> Capacitor_SMD:C_0402_1005Metric
- C31: renamed from C26; footprint (none) -> Capacitor_SMD:C_0402_1005Metric
- C32: renamed from C28; footprint (none) -> Capacitor_SMD:C_0402_1005Metric
- C33: renamed from C27; footprint (none) -> Capacitor_SMD:C_0402_1005Metric
- C34: renamed from C30; footprint (none) -> Capacitor_SMD:C_0402_1005Metric
- C35: renamed from C29; footprint (none) -> Capacitor_SMD:C_0402_1005Metric
- FB2: renamed from FB1; footprint (none) -> Inductor_SMD:L_0603_1608Metric
- FB3: renamed from FB2; footprint (none) -> Inductor_SMD:L_0603_1608Metric
- R18: renamed from R15; footprint (none) -> Resistor_SMD:R_0402_1005Metric
- R19: renamed from R11; footprint (none) -> Resistor_SMD:R_0402_1005Metric
- R20: renamed from R12; footprint (none) -> Resistor_SMD:R_0402_1005Metric
- R21: renamed from R13; footprint (none) -> Resistor_SMD:R_0402_1005Metric
- R22: renamed from R14; footprint (none) -> Resistor_SMD:R_0402_1005Metric
- renumbered TP11 to TP1, TP8 to TP10, TP9 to TP11, TP10 to TP12, TP12 to TP2, TP1 to TP3, TP2 to TP4, TP3 to TP5, TP4 to TP6, TP5 to TP7, TP6 to TP8, TP7 to TP9, U1 to U8

Commit message: add images and render
Parts:
- added C36: 4.7uF, Capacitor_SMD:C_0402_1005Metric, symbol Device:C_Small
- TP1, TP10, TP11, TP12, TP2, TP3, TP4, TP5, TP6, TP7, TP8, TP9: now left out of the parts list
Connections:
- net GND: now also C36.2
- net VBUS: now reaches U8.40 (VREGIN)
- net VBUS: now also C36.1
Changed lines of the file:
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@@
 	)
 	(junction
+		(at 55.88 60.96)
+		(diameter 0)
+		(color 0 0 0 0)
+	)
+	(junction
 		(at 100.33 130.81)
 		(diameter 0)
@@
 	(wire
 		(pts
+			(xy 53.34 60.96) (xy 55.88 60.96)
+		)
+		(stroke
+			(width 0)
+			(type default)
+		)
+	)
+	(wire
+		(pts
 			(xy 92.71 41.91) (xy 95.25 41.91)
 		)
@@
 	(wire
 		(pts
+			(xy 55.88 60.96) (xy 69.85 60.96)
+		)
+		(stroke
+			(width 0)
+			(type default)
+		)
+	)
+	(wire
+		(pts
 			(xy 123.19 149.86) (xy 124.46 149.86)
 		)
@@
 		)
 	)
+	(wire
+		(pts
+			(xy 55.88 66.04) (xy 55.88 67.31)
+		)
+		(stroke
+			(width 0)
+			(type default)
+		)
+	)
 	(global_label "VPLL"
 		(shape input)
@@
 		)
 	)
+	(hierarchical_label "VBUS"
+		(shape input)
+		(at 53.34 60.96 180)
+		(effects
+			(font
+				(size 1.27 1.27)
+			)
+			(justify right)
+		)
+	)
 	(hierarchical_label "3.3V"
 		(shape input)
@@
 		(body_style 1)
 		(exclude_from_sim no)
-		(in_bom yes)
+		(in_bom no)
 		(on_board yes)
 		(in_pos_files yes)
@@
 		(body_style 1)
 		(exclude_from_sim no)
-		(in_bom yes)
+		(in_bom no)
 		(on_board yes)
 		(in_pos_files yes)
@@
 		(body_style 1)
 		(exclude_from_sim no)
-		(in_bom yes)
+		(in_bom no)
 		(on_board yes)
 		(in_pos_files yes)
@@
 		(body_style 1)
 		(exclude_from_sim no)
-		(in_bom yes)
+		(in_bom no)
 		(on_board yes)
 		(in_pos_files yes)
@@
 	(symbol
 		(lib_id "power:GND")
+		(at 55.88 67.31 0)
+		(unit 1)
+		(body_style 1)
+		(exclude_from_sim no)
+		(in_bom yes)
+		(on_board yes)
+		(in_pos_files yes)
+		(dnp no)
+		(fields_autoplaced yes)
+		(property "Reference" "#PWR042"
+			(at 55.88 73.66 0)
+			(hide yes)
+			(show_name no)
+			(do_not_autoplace no)
+			(effects
+				(font
+					(size 1.27 1.27)
+				)
+			)
+		)
+		(property "Value" "GND"
+			(at 55.88 72.39 0)
+			(show_name no)
+			(do_not_autoplace no)
+			(effects
+				(font
+					(size 1.27 1.27)
+				)
+			)
+		)
+		(property "Footprint" ""
+			(at 55.88 67.31 0)
+			(hide yes)
+			(show_name no)
+			(do_not_autoplace no)
+			(effects
+				(font
+					(size 1.27 1.27)
+				)
+			)
+		)
+		(property "Datasheet" ""
+			(at 55.88 67.31 0)
+			(hide yes)
+			(show_name no)
+			(do_not_autoplace no)
+			(effects
+				(font
+					(size 1.27 1.27)
+				)
+			)
+		)
+		(property "Description" "Power symbol creates a global label with name \"GND\" , ground"
+			(at 55.88 67.31 0)
+			(hide yes)
+			(show_name no)
+			(do_not_autoplace no)
+			(effects
+				(font
+					(size 1.27 1.27)
+				)
+			)
+		)
+		(pin "1"
+		)
+		(instances
+			(project "FPGA_Board"
+				(path "/ed5fd1e9-0492-49f2-b736-bd16e22cfa0b/9842cdb2-2418-485e-9db8-b113a4b99c71"
+					(reference "#PWR042")
+					(unit 1)
+				)
+			)
+		)
+	)
+	(symbol
+		(lib_id "power:GND")
 		(at 93.98 132.08 0)
 		(unit 1)
@@
 		(body_style 1)
 		(exclude_from_sim no)
-		(in_bom yes)
+		(in_bom no)
 		(on_board yes)
 		(in_pos_files yes)
@@
 		(body_style 1)
 		(exclude_from_sim no)
-		(in_bom yes)
+		(in_bom no)
 		(on_board yes)
 		(in_pos_files yes)
@@
 	(symbol
 		(lib_id "Device:C_Small")
+		(at 55.88 63.5 0)
+		(unit 1)
+		(body_style 1)
+		(exclude_from_sim no)
+		(in_bom yes)
+		(on_board yes)
+		(in_pos_files yes)
+		(dnp no)
+		(fields_autoplaced yes)
+		(property "Reference" "C36"
+			(at 58.42 62.2362 0)
+			(show_name no)
+			(do_not_autoplace no)
+			(effects
+				(font
+					(size 1.27 1.27)
+				)
+				(justify left)
+			)
+		)
+		(property "Value" "4.7uF"
+			(at 58.42 64.7762 0)
+			(show_name no)
+			(do_not_autoplace no)
+			(effects
+				(font
+					(size 1.27 1.27)
+				)
+				(justify left)
+			)
+		)
+		(property "Footprint" "Capacitor_SMD:C_0402_1005Metric"
+			(at 55.88 63.5 0)
+			(hide yes)
+			(show_name no)
+			(do_not_autoplace no)
+			(effects
+				(font
+					(size 1.27 1.27)
+				)
+			)
+		)
+		(property "Datasheet" ""
+			(at 55.88 63.5 0)
+			(hide yes)
+			(show_name no)
+			(do_not_autoplace no)
+			(effects
+				(font
+					(size 1.27 1.27)
+				)
+			)
+		)
+		(property "Description" "Unpolarized capacitor, small symbol"
+			(at 55.88 63.5 0)
+			(hide yes)
+			(show_name no)
+			(do_not_autoplace no)
+			(effects
+				(font
+					(size 1.27 1.27)
+				)
+			)
+		)
+		(pin "2"
+		)
+		(pin "1"
+		)
+		(instances
+			(project "FPGA_Board"
+				(path "/ed5fd1e9-0492-49f2-b736-bd16e22cfa0b/9842cdb2-2418-485e-9db8-b113a4b99c71"
+					(reference "C36")
+					(unit 1)
+				)
+			)
+		)
+	)
+	(symbol
+		(lib_id "Device:C_Small")
 		(at 130.81 45.72 0)
 		(unit 1)
@@
 		(body_style 1)
 		(exclude_from_sim no)
-		(in_bom yes)
+		(in_bom no)
 		(on_board yes)
 		(in_pos_files yes)
@@
 		(body_style 1)
 		(exclude_from_sim no)
-		(in_bom yes)
+		(in_bom no)
 		(on_board yes)
 		(in_pos_files yes)
@@
 		(body_style 1)
 		(exclude_from_sim no)
-		(in_bom yes)
+		(in_bom no)
 		(on_board yes)
 		(in_pos_files yes)
@@
 		(body_style 1)
 		(exclude_from_sim no)
-		(in_bom yes)
+		(in_bom no)
 		(on_board yes)
 		(in_pos_files yes)
@@
 		(body_style 1)
 		(exclude_from_sim no)
-		(in_bom yes)
+		(in_bom no)
 		(on_board yes)
 		(in_pos_files yes)
@@
 		(body_style 1)
 		(exclude_from_sim no)
-		(in_bom yes)
+		(in_bom no)
 		(on_board yes)
 		(in_pos_files yes)

Commit message: update bom and journal
Parts:
- added C38: 0.1uF, Capacitor_SMD:C_0402_1005Metric, symbol Device:C_Small
Connections:
- net 3.3V: now also C38.1
- net GND: now also C38.2
Other:
- moved on the sheet: R19, R20, R21, R22, U9

Commit message: journal
Changed lines of the file:
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@@
+		)
+	)
+	(label "3.3V"
+		(at 120.65 41.91 0)
+		(effects
+			(font
+				(size 1.27 1.27)
+			)
+			(justify left bottom)
+		)
+	)
+	(label "3.3V"
+		(at 138.43 140.97 0)
+		(effects
+			(font
+				(size 1.27 1.27)
+			)
+			(justify left bottom)
 		)
 	)
