File: kicad/FPGA_Board.kicad_pcb (KiCad board)
At the start: 2 copper layers, 50 x 70 mm, 0 parts

Commit message: finish schematic and almost done pcb routing
Parts:
- added C1: 10uF, Capacitor_SMD:C_0402_1005Metric, F.Cu at (72.0, 100.0)
- added C10: 0.1uF, Capacitor_SMD:C_0402_1005Metric, F.Cu at (83.0, 97.0)
- added C11: 0.1uF, Capacitor_SMD:C_0402_1005Metric, F.Cu at (83.0, 95.0)
- added C12: 10uF, Capacitor_SMD:C_0402_1005Metric, F.Cu at (83.0, 91.0)
- added C13: 10uF, Capacitor_SMD:C_0402_1005Metric, F.Cu at (83.0, 99.0)
- added C14: 10uF, Capacitor_SMD:C_0402_1005Metric, F.Cu at (83.0, 93.0)
- added C15: 0.1uF, Capacitor_SMD:C_0402_1005Metric, F.Cu at (50.0, 75.0)
- added C16: 0.1uF, Capacitor_SMD:C_0402_1005Metric, F.Cu at (61.2, 72.1)
- added C17: 10uF, Capacitor_SMD:C_0402_1005Metric, F.Cu at (107.3, 59.7)
- added C18: 0.1uF, Capacitor_SMD:C_0402_1005Metric, F.Cu at (57.5, 64.5)
- added C19: 0.1uF, Capacitor_SMD:C_0402_1005Metric, F.Cu at (71.4, 66.4)
- added C2: 10uF, Capacitor_SMD:C_0402_1005Metric, F.Cu at (72.0, 104.0)
- added C20: 0.1uF, Capacitor_SMD:C_0402_1005Metric, F.Cu at (70.0, 63.1)
- added C21: 0.1uF, Capacitor_SMD:C_0402_1005Metric, F.Cu at (57.5, 66.8)
- added C22: 0.1uF, Capacitor_SMD:C_0402_1005Metric, F.Cu at (59.6, 70.0)
- added C23: 0.1uF, Capacitor_SMD:C_0402_1005Metric, F.Cu at (57.9, 69.5)
- added C24: 10uF, Capacitor_SMD:C_0402_1005Metric, F.Cu at (60.8, 52.3)
- added C25: 0.1uF, Capacitor_SMD:C_0402_1005Metric, F.Cu at (60.1, 51.6)
- added C26: 0.1uF, Capacitor_SMD:C_0402_1005Metric, F.Cu at (52.0, 79.0)
- added C27: 0.1uF, Capacitor_SMD:C_0402_1005Metric, F.Cu at (58.0, 84.0)
- added C28: 0.1uF, Capacitor_SMD:C_0402_1005Metric, F.Cu at (58.0, 83.0)
- added C29: 0.1uF, Capacitor_SMD:C_0402_1005Metric, F.Cu at (68.2, 92.0)
- added C3: 10uF, Capacitor_SMD:C_0402_1005Metric, F.Cu at (77.0, 91.0)
- added C30: 0.1uF, Capacitor_SMD:C_0402_1005Metric, F.Cu at (71.0, 83.0)
- added C31: 0.1uF, Capacitor_SMD:C_0402_1005Metric, F.Cu at (59.0, 89.0)
- added C32: 0.1uF, Capacitor_SMD:C_0402_1005Metric, F.Cu at (63.0, 93.0)
- added C33: 0.1uF, Capacitor_SMD:C_0402_1005Metric, F.Cu at (66.3, 92.0)
- added C34: 10uF, Capacitor_SMD:C_0402_1005Metric, F.Cu at (62.0, 93.0)
- added C35: 10uF, Capacitor_SMD:C_0402_1005Metric, F.Cu at (66.3, 93.0)
- added C4: 10uF, Capacitor_SMD:C_0402_1005Metric, F.Cu at (77.0, 97.0)
- added C5: 10uF, Capacitor_SMD:C_0402_1005Metric, F.Cu at (77.0, 93.0)
- added C6: 0.1uF, Capacitor_SMD:C_0402_1005Metric, F.Cu at (77.0, 89.0)
- added C7: 0.1uF, Capacitor_SMD:C_0402_1005Metric, F.Cu at (77.0, 99.0)
- added C8: 0.1uF, Capacitor_SMD:C_0402_1005Metric, F.Cu at (77.0, 95.0)
- added C9: 0.1uF, Capacitor_SMD:C_0402_1005Metric, F.Cu at (83.0, 89.0)
- added D1: LED_ARGB, LED_SMD:LED_Cree-PLCC4_2x2mm_CW, F.Cu at (110.3, 59.7)
- added D2: GREEN, LED_SMD:LED_0402_1005Metric, F.Cu at (110.8, 67.9)
- added FB1: BLM18HE152SN1D, Inductor_SMD:L_0603_1608Metric, F.Cu at (72.0, 102.0)
- added FB2: BLM18HE152SN1D, Inductor_SMD:L_0603_1608Metric, F.Cu at (60.0, 93.0)
- added FB3: BLM18HE152SN1D, Inductor_SMD:L_0603_1608Metric, F.Cu at (69.0, 94.0)
- added FID1: Fiducial, Fiducial:Fiducial_0.5mm_Mask1mm, F.Cu at (47.0, 41.0)
- added FID2: Fiducial, Fiducial:Fiducial_0.5mm_Mask1mm, F.Cu at (88.0, 49.0)
- added FID3: Fiducial, Fiducial:Fiducial_0.5mm_Mask1mm, F.Cu at (88.0, 101.0)
- added FID4: Fiducial, Fiducial:Fiducial_0.5mm_Mask1mm, F.Cu at (42.0, 101.0)
- added FID5: Fiducial, Fiducial:Fiducial_Cross_1.5mm_Mask2mm, F.Cu at (65.0, 106.1)
- added H1: MountingHole, MountingHole:MountingHole_3.2mm_M3, F.Cu at (45.0, 45.0)
- added H2: MountingHole, MountingHole:MountingHole_3.2mm_M3, F.Cu at (85.0, 45.0)
- added H3: MountingHole, MountingHole:MountingHole_3.2mm_M3, F.Cu at (85.0, 105.0)
- added H4: MountingHole, MountingHole:MountingHole_3.2mm_M3, F.Cu at (45.0, 105.0)
- added J1: USB_C_Receptacle_USB2.0_14P, Connector_USB:USB_C_Receptacle_HRO_TYPE-C-31-M-12, F.Cu at (65.0, 106.1)
- added J3: Conn_02x12_Odd_Even, Connector_PinHeader_2.54mm:PinHeader_2x12_P2.54mm_Vertical, F.Cu at (43.7, 51.0)
- added J4: Conn_02x12_Odd_Even, Connector_PinHeader_2.54mm:PinHeader_2x12_P2.54mm_Vertical, F.Cu at (82.7, 51.0)
- added R1: 5.1k, Resistor_SMD:R_0402_1005Metric, F.Cu at (69.0, 100.0)
- added R10: 10k, Resistor_SMD:R_0402_1005Metric, F.Cu at (61.5, 53.1)
- added R11: 10k, Resistor_SMD:R_0402_1005Metric, F.Cu at (53.0, 60.8)
- added R12: 100, Resistor_SMD:R_0402_1005Metric, F.Cu at (60.3, 70.7)
- added R13: 0, Resistor_SMD:R_0402_1005Metric, F.Cu at (58.0, 79.0)
- added R14: 0R, Resistor_SMD:R_0402_1005Metric, F.Cu at (59.0, 75.0)
- added R15: 0R, Resistor_SMD:R_0402_1005Metric, F.Cu at (64.9, 59.6)
- added R16: 0R, Resistor_SMD:R_0402_1005Metric, F.Cu at (59.8, 63.5)
- added R17: 0R, Resistor_SMD:R_0402_1005Metric, F.Cu at (64.2, 58.9)
- added R18: 12k, Resistor_SMD:R_0402_1005Metric, F.Cu at (64.0, 93.0)
- added R19: 10k, Resistor_SMD:R_0402_1005Metric, F.Cu at (51.2, 92.0)
- added R2: 5.1k, Resistor_SMD:R_0402_1005Metric, F.Cu at (61.0, 100.0)
- added R20: 10k, Resistor_SMD:R_0402_1005Metric, F.Cu at (51.0, 82.0)
- added R21: 10k, Resistor_SMD:R_0402_1005Metric, F.Cu at (55.0, 82.0)
- added R22: 2.2k, Resistor_SMD:R_0402_1005Metric, F.Cu at (53.0, 82.0)
- added R3: 5.1k, Resistor_SMD:R_0402_1005Metric, F.Cu at (68.0, 98.0)
- added R4: 5.1k, Resistor_SMD:R_0402_1005Metric, F.Cu at (62.0, 98.0)
- added R5: 10k, Resistor_SMD:R_0402_1005Metric, F.Cu at (68.6, 61.7)
- added R6: 10k, Resistor_SMD:R_0402_1005Metric, F.Cu at (70.0, 60.4)
- added R7: 1k, Resistor_SMD:R_0402_1005Metric, F.Cu at (108.8, 67.9)
- added R8: 0R, Resistor_SMD:R_0402_1005Metric, F.Cu at (62.2, 53.8)
- added R9: 0R, Resistor_SMD:R_0402_1005Metric, F.Cu at (53.8, 62.2)
- added SW1: SW_Push, Button_Switch_SMD:Panasonic_EVQPUM_EVQPUD, F.Cu at (65.0, 42.0)
- added TP1: TestPoint, TestPoint:TestPoint_Pad_1.0x1.0mm, F.Cu at (72.0, 77.0)
- added TP10: TestPoint, TestPoint:TestPoint_Pad_1.0x1.0mm, F.Cu at (64.0, 79.0)
- added TP11: TestPoint, TestPoint:TestPoint_Pad_1.0x1.0mm, F.Cu at (62.0, 77.0)
- added TP12: TestPoint, TestPoint:TestPoint_Pad_1.0x1.0mm, F.Cu at (62.0, 79.0)
- added TP2: TestPoint, TestPoint:TestPoint_Pad_1.0x1.0mm, F.Cu at (72.0, 79.0)
- added TP3: TestPoint, TestPoint:TestPoint_Pad_1.0x1.0mm, F.Cu at (70.0, 77.0)
- added TP4: TestPoint, TestPoint:TestPoint_Pad_1.0x1.0mm, F.Cu at (70.0, 79.0)
- added TP5: TestPoint, TestPoint:TestPoint_Pad_1.0x1.0mm, F.Cu at (68.0, 77.0)
- added TP6: TestPoint, TestPoint:TestPoint_Pad_1.0x1.0mm, F.Cu at (68.0, 79.0)
- added TP7: TestPoint, TestPoint:TestPoint_Pad_1.0x1.0mm, F.Cu at (66.0, 77.0)
- added TP8: TestPoint, TestPoint:TestPoint_Pad_1.0x1.0mm, F.Cu at (66.0, 79.0)
- added TP9: TestPoint, TestPoint:TestPoint_Pad_1.0x1.0mm, F.Cu at (64.0, 77.0)
- added U1: USBLC6-2SC6, Package_TO_SOT_SMD:SOT-23-6, F.Cu at (65.0, 98.0)
- added U2: TLV75712PDBV, Package_TO_SOT_SMD:SOT-23-5, F.Cu at (80.0, 90.0)
- added U3: TLV75725PDBV, Package_TO_SOT_SMD:SOT-23-5, F.Cu at (80.0, 98.0)
- added U4: TLV75733PDBV, Package_TO_SOT_SMD:SOT-23-5, F.Cu at (80.0, 94.0)
- added U5: 74AUC2G240, Package_SO:VSSOP-8_3x3mm_P0.65mm, F.Cu at (55.0, 74.0)
- added U6: ICE40UP5K-SG48ITR, Package_DFN_QFN:QFN-48-1EP_7x7mm_P0.5mm_EP5.6x5.6mm, F.Cu at (65.1, 66.7)
- added U7: W25Q128JVS, Package_SO:SOIC-8_5.3x5.3mm_P1.27mm, F.Cu at (58.0, 58.0)
- added U8: FT232H, Package_QFP:LQFP-48_7x7mm_P0.5mm, F.Cu at (65.0, 86.0)
- added U9: 93LC56BT-I/OT, Package_SO:SOIC-8_3.9x4.9mm_P1.27mm, F.Cu at (53.0, 87.0)
- added Y1: SG-210STF, Oscillator:Oscillator_SMD_SeikoEpson_SG210-4Pin_2.5x2.0mm, F.Cu at (55.0, 78.0)
Routing:
- net /FPGA/IOB_18a: track 0.00 -> 54.3 mm, vias 0 -> 1
- net /FPGA/1.2V: track 0.00 -> 52.6 mm, vias 0 -> 3
- net /Clock/IOB_25b_G3: track 0.00 -> 52.1 mm, vias 0 -> 3
- net /Config/USB_D+: track 0.00 -> 52.0 mm, vias 0 -> 3
- net /Clock/3.3V: track 0.00 -> 51.2 mm, vias 0 -> 15
- net /FPGA/CDONE: track 0.00 -> 50.5 mm, vias 0 -> 2
- net /FPGA/2.5V: track 0.00 -> 49.6 mm, vias 0 -> 2
- net /Config/USB_D-: track 0.00 -> 44.7 mm, vias 0 -> 2
- net /FPGA/CRESET: track 0.00 -> 44.3 mm, vias 0 -> 2
- net /FPGA/FPGA_SO: track 0.00 -> 41.7 mm, vias 0 -> 1
- net /FPGA/FT_SCK: track 0.00 -> 41.5 mm, vias 0 -> 1
- net /FPGA/FT_CS: track 0.00 -> 39.2 mm, vias 0 -> 1
- net /Power/VIN: track 0.00 -> 37.4 mm
- net /FPGA/FPGA_SI: track 0.00 -> 34.4 mm, vias 0 -> 1
- net /Config/IOB_24a: track 0.00 -> 31.8 mm
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- added copper zone on In2.Cu, net /Clock/3.3V
- added copper zone on F.Cu, net GND
- added copper zone on In1.Cu, net GND
Other:
- copper layers 2 -> 4

Commit message: add images and render
Parts:
- removed FID5: Fiducial, Fiducial:Fiducial_Cross_1.5mm_Mask2mm
- added C36: 4.7uF, Capacitor_SMD:C_0402_1005Metric, F.Cu at (58.0, 85.0)
- added G***: LOGO, logo:linuxpenguin_cu, F.Cu at (55.0, 102.5)
- added G***: LOGO, logo:linuxpenguin-mask, F.Cu at (55.0, 102.5)
- added TP13: TestPoint, TestPoint:TestPoint_Pad_2.0x2.0mm, F.Cu at (85.0, 90.0)
- added TP14: TestPoint, TestPoint:TestPoint_Pad_2.0x2.0mm, F.Cu at (85.0, 98.0)
- added TP15: TestPoint, TestPoint:TestPoint_Pad_2.0x2.0mm, F.Cu at (85.0, 94.0)
- moved C17 55.5 mm to (54.5, 42.5)
- moved D1 55.5 mm to (57.5, 42.5)
- moved D2 48.0 mm to (70.0, 42.5), turned to -90 degrees
- moved R7 45.3 mm to (70.0, 44.5), turned to 90 degrees
- moved C26 3.29 mm to (55.0, 80.3), turned to 0 degrees
Connections:
- U8 pad 40: unconnected-(U8-VREGIN-Pad40) -> /Flasher/VBUS
Routing:
- net /FPGA/RGB1: track 17.7 -> 71.6 mm, vias 0 -> 1
- net /FPGA/RGB2: track 20.0 -> 67.1 mm, vias 0 -> 1
- net /FPGA/RGB0: track 21.4 -> 65.7 mm, vias 0 -> 1
- net /FPGA/FT_CS: track 39.2 -> 83.3 mm, vias 1 -> 2
- net /FPGA/FPGA_SI: track 34.4 -> 72.6 mm, vias 1 -> 2
- net /FPGA/FT_SCK: track 41.5 -> 76.2 mm, vias 1 -> 2
- net /FPGA/FPGA_SO: track 41.7 -> 74.5 mm, vias 1 -> 2
- net /FPGA/CRESET: track 44.3 -> 70.5 mm, vias 2 -> 3
- net /FPGA/CDONE: track 50.5 -> 69.2 mm, vias 2 -> 3
- net /Clock/3.3V: track 51.2 -> 65.0 mm, vias 15 -> 14
- net /Flasher/VBUS: track 0.00 -> 2.46 mm
- net Net-(D2-A): track 0.00 -> 1.01 mm
- net /FPGA/IOB_18a: track 54.3 -> 55.2 mm
- net GND: vias 28 -> 29
Other:
- board text added: "0a 5b"
- board text added: "1.2V"
- board text added: "13 8a"
- board text added: "18 16"
- board text added: "2.5V"
- board text added: "22 20"
- board text added: "23 37"
- board text added: "24 32"
- board text added: "29 25"
- board text added: "3.3V"
- board text added: "3.3v G"
- board text added: "33 31"
- board text added: "34 35"
- board text added: "36 39"
- board text added: "38 41"
- board text added: "3b 49"
- board text added: "42 43"
- board text added: "44 46"
- board text added: "48 M"
- board text added: "4a 2a"
- board text added: "50 45"
- board text added: "51 R2"
- board text added: "9b 6a"
- board text added: "CDONE"
- board text added: "CRESET"
- board text added: "Converts Bitcoins into Dreams."
- board text added: "G 3.3v"
- board text added: "GN GN"
- board text added: "R1 R0"
- board text added: "RS DN"

Commit message: update bom and journal
Parts:
- added C37: 0.1uF, Capacitor_SMD:C_0402_1005Metric, F.Cu at (61.8, 94.9)
- added C38: 0.1uF, Capacitor_SMD:C_0402_1005Metric, F.Cu at (53.6, 92.0)
- added R23: 10k, Resistor_SMD:R_0402_1005Metric, F.Cu at (78.4, 81.5)
- added R24: 10k, Resistor_SMD:R_0402_1005Metric, F.Cu at (78.4, 83.9)
- R3, R4: value 5.1k -> 22
Connections:
- U3 pad 3: /Power/VIN -> /FPGA/1.2V
- U4 pad 3: /Power/VIN -> /FPGA/2.5V
Routing:
- net /FPGA/1.2V: track 52.6 -> 63.2 mm, vias 3 -> 5
- net /Clock/3.3V: track 65.0 -> 70.9 mm, vias 14 -> 15
- net /FPGA/FT_SCK: track 76.2 -> 80.5 mm, vias 2 -> 3
- net /Power/VIN: track 37.4 -> 33.3 mm
- net Net-(U1-VBUS): track 18.3 -> 21.9 mm, vias 4 -> 5
- net /FPGA/2.5V: track 49.6 -> 51.3 mm, vias 2 -> 3
- net GND: vias 29 -> 30

Commit message: journal
Routing:
- net /Config/USB_D+: track 52.0 -> 60.2 mm
- net GND: track 19.4 -> 24.0 mm
- net /Config/USB_D-: track 44.7 -> 46.6 mm
- net /FPGA/2.5V: track 51.3 -> 53.0 mm
- net /FPGA/FPGA_SI: track 72.6 -> 73.1 mm

Commit message: journal
Parts:
- U6: footprint Package_DFN_QFN:QFN-48-1EP_7x7mm_P0.5mm_EP5.6x5.6mm -> Package_DFN_QFN:QFN-48-1EP_7x7mm_P0.5mm_EP3.5x3.5mm_ThermalVias
Connections:
- net /Clock/3.3V renamed /Flasher/3.3V
Routing:
- net GND: track 24.0 -> 44.8 mm, vias 30 -> 49
- net /Flasher/3.3V: track 70.9 -> 79.3 mm, vias 15 -> 17
- net /FPGA/CDONE: track 69.2 -> 77.1 mm
- net Net-(U1-VBUS): track 21.9 -> 27.7 mm
- net /FPGA/1.2V: track 63.2 -> 65.5 mm
- net /FPGA/RGB1: track 71.6 -> 73.8 mm
- net /Clock/IOB_25b_G3: track 52.1 -> 54.2 mm
- net /FPGA/RGB2: track 67.1 -> 68.9 mm
- net /FPGA/2.5V: track 53.0 -> 54.5 mm
- net /FPGA/FPGA_SI: track 73.1 -> 72.3 mm
