File: kicad/fpga.kicad_sch (KiCad schematic)
At the start: 23 parts, among them SW1 SW_Push, U6 ICE40UP5K-SG48ITR, U7 W25Q128JVS

Commit message: finish schematic and almost done pcb routing
Parts:
- C16: renamed from C15; footprint (none) -> Capacitor_SMD:C_0402_1005Metric
- C17: renamed from C23; footprint (none) -> Capacitor_SMD:C_0402_1005Metric
- C18: renamed from C16; footprint (none) -> Capacitor_SMD:C_0402_1005Metric
- C19: renamed from C17; footprint (none) -> Capacitor_SMD:C_0402_1005Metric
- C20: renamed from C18; footprint (none) -> Capacitor_SMD:C_0402_1005Metric
- C21: renamed from C19; footprint (none) -> Capacitor_SMD:C_0402_1005Metric
- C22: renamed from C20; footprint (none) -> Capacitor_SMD:C_0402_1005Metric
- C23: renamed from C35; footprint (none) -> Capacitor_SMD:C_0402_1005Metric
- C24: renamed from C21; footprint (none) -> Capacitor_SMD:C_0402_1005Metric
- C25: renamed from C22; footprint (none) -> Capacitor_SMD:C_0402_1005Metric
- D1: renamed from D2; footprint (none) -> LED_SMD:LED_Cree-PLCC4_2x2mm_CW
- D2: renamed from D1; footprint (none) -> LED_SMD:LED_0402_1005Metric
- R10: renamed from R8; footprint (none) -> Resistor_SMD:R_0402_1005Metric
- R11: renamed from R9; footprint (none) -> Resistor_SMD:R_0402_1005Metric
- R12: renamed from R22; footprint (none) -> Resistor_SMD:R_0402_1005Metric
- R5, R6, R7: footprint (none) -> Resistor_SMD:R_0402_1005Metric
- R8: renamed from R20; footprint (none) -> Resistor_SMD:R_0402_1005Metric
- R9: renamed from R19; footprint (none) -> Resistor_SMD:R_0402_1005Metric
- SW1: footprint (none) -> Button_Switch_SMD:Panasonic_EVQPUM_EVQPUD
Connections:
- net +3.3V is gone; now on net 3.3V: C24.1, C25.1, R10.1, R11.1, U7.8 (VCC)

Commit message: update bom and journal
Parts:
- added R23, R24: 10k, Resistor_SMD:R_0402_1005Metric, symbol Device:R_Small_US
Connections:
- net 3.3V: now also R23.1, R24.1
- net FT_CS: now also R23.2
- net FT_SCK: now also R24.2
Other:
- moved on the sheet: R10, R11, R8, R9

Commit message: journal
Parts:
- U6: footprint Package_DFN_QFN:QFN-48-1EP_7x7mm_P0.5mm_EP5.6x5.6mm -> Package_DFN_QFN:QFN-48-1EP_7x7mm_P0.5mm_EP3.5x3.5mm
Changed lines of the file:
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@@
 			)
 		)
-		(property "Footprint" "Package_DFN_QFN:QFN-48-1EP_7x7mm_P0.5mm_EP5.6x5.6mm"
+		(property "Footprint" "Package_DFN_QFN:QFN-48-1EP_7x7mm_P0.5mm_EP3.5x3.5mm"
 			(at 130.81 120.65 0)
 			(hide yes)
@@
 			)
 		)
-		(property "Footprint" "Package_DFN_QFN:QFN-48-1EP_7x7mm_P0.5mm_EP5.6x5.6mm"
+		(property "Footprint" "Package_DFN_QFN:QFN-48-1EP_7x7mm_P0.5mm_EP3.5x3.5mm"
 			(at 67.31 120.65 0)
 			(hide yes)
@@
 			)
 		)
-		(property "Footprint" "Package_DFN_QFN:QFN-48-1EP_7x7mm_P0.5mm_EP5.6x5.6mm"
+		(property "Footprint" "Package_DFN_QFN:QFN-48-1EP_7x7mm_P0.5mm_EP3.5x3.5mm"
 			(at 168.91 120.65 0)
 			(hide yes)
@@
 			)
 		)
-		(property "Footprint" "Package_DFN_QFN:QFN-48-1EP_7x7mm_P0.5mm_EP5.6x5.6mm"
+		(property "Footprint" "Package_DFN_QFN:QFN-48-1EP_7x7mm_P0.5mm_EP3.5x3.5mm"
 			(at 219.71 120.65 0)
 			(hide yes)

Commit message: journal
Parts:
- U6: footprint Package_DFN_QFN:QFN-48-1EP_7x7mm_P0.5mm_EP3.5x3.5mm -> Package_DFN_QFN:QFN-48-1EP_7x7mm_P0.5mm_EP3.5x3.5mm_ThermalVias
Changed lines of the file:
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@@
 			)
 		)
-		(property "Footprint" "Package_DFN_QFN:QFN-48-1EP_7x7mm_P0.5mm_EP3.5x3.5mm"
+		(property "Footprint" "Package_DFN_QFN:QFN-48-1EP_7x7mm_P0.5mm_EP3.5x3.5mm_ThermalVias"
 			(at 130.81 120.65 0)
 			(hide yes)
@@
 			)
 		)
-		(property "Footprint" "Package_DFN_QFN:QFN-48-1EP_7x7mm_P0.5mm_EP3.5x3.5mm"
+		(property "Footprint" "Package_DFN_QFN:QFN-48-1EP_7x7mm_P0.5mm_EP3.5x3.5mm_ThermalVias"
 			(at 67.31 120.65 0)
 			(hide yes)
@@
 			)
 		)
-		(property "Footprint" "Package_DFN_QFN:QFN-48-1EP_7x7mm_P0.5mm_EP3.5x3.5mm"
+		(property "Footprint" "Package_DFN_QFN:QFN-48-1EP_7x7mm_P0.5mm_EP3.5x3.5mm_ThermalVias"
 			(at 168.91 120.65 0)
 			(hide yes)
@@
 			)
 		)
-		(property "Footprint" "Package_DFN_QFN:QFN-48-1EP_7x7mm_P0.5mm_EP3.5x3.5mm"
+		(property "Footprint" "Package_DFN_QFN:QFN-48-1EP_7x7mm_P0.5mm_EP3.5x3.5mm_ThermalVias"
 			(at 219.71 120.65 0)
 			(hide yes)
